Commit message: Gazebo Simulation almost up and running

File: description/gazebo_control.xacro (robot description, xacro)
@@ -3,4 +3,5 @@
     <gazebo>
         <plugin name="gz::sim::systems::DiffDrive" filename="gz-sim-diff-drive-system">
+            <alwaysOn>true</alwaysOn>
             <!-- Wheel info -->
             <left_joint>left_wheel_joint</left_joint>
@@ -11,13 +12,11 @@
             <max_wheel_torque>200</max_wheel_torque>
             <max_wheel_acceleration>10.0</max_wheel_acceleration>
+            <topic>cmd_vel</topic>
             <!-- Output -->
-            <odometry_frame>odom</odometry_frame>
-            <robot_base_frame>base_link</robot_base_frame>
+            <robotBaseFrame>base_link</robotBaseFrame>
             <odom_publish_frequency>1</odom_publish_frequency>
             <publish_odom>true</publish_odom>
-            <odom_publish_frequency>1</odom_publish_frequency>
             <publish_odom_tf>true</publish_odom_tf>
             <publish_wheel_tf>true</publish_wheel_tf>
-            <topic>cmd_vel</topic>
         </plugin>
         <!-- Moving Forward-->
@@ -58,4 +57,22 @@
             </output>
         </plugin>
+        <plugin
+            filename="gz-sim-joint-state-publisher-system"
+            name="gz::sim::systems::JointStatePublisher">
+        </plugin>
+        <plugin
+            filename="gz-sim-pose-publisher-system"
+            name="gz::sim::systems::PosePublisher">
+            <!-- <publish_link_pose>true</publish_link_pose> -->
+            <!-- <use_pose_vector_msg>true</use_pose_vector_msg> -->
+            <static_publisher>true</static_publisher>
+            <static_update_frequency>1</static_update_frequency>
+        </plugin>
+        <plugin
+            filename="gz-sim-odometry-publisher-system"
+            name="gz::sim::systems::OdometryPublisher">
+            <odom_frame>odom</odom_frame>
+            <robot_base_frame>botwheel</robot_base_frame>
+        </plugin>
     </gazebo>
 </robot>

File: description/lidar.xacro (robot description, xacro)
@@ -16,5 +16,5 @@
             <geometry>
                 <cylinder radius="0.08" length="0.045"/>
-            </geometry>
+            </geometry>f
         </collision>
         <xacro:inertial_cylinder mass="0.15" length="0.04" radius="0.05">
@@ -45,8 +45,12 @@
                 </range>
             </ray>
-            <plugin name="laser_controller" filename="gz-sim-sensors-system">
+            <!-- <plugin name="laser_controller" filename="gz-sim-sensors-system">
+                <ros>
+                    <argument>~/out:=scan</argument>
+                </ros>
                 <output_type>sensor_msgs/LaserScan</output_type>
                 <frame_name>laser_frame</frame_name>
-            </plugin>
+            </plugin> -->
+            <gz_frame_id>laser_frame</gz_frame_id>
         </sensor>
     </gazebo>

File: description/model.urdf (robot description, URDF)
Before this commit: robot robot, 6 links, 5 joints
Links:
- removed link base_link
- added link botwheel
- added link camera_link; visual box size=0.010 0.03 0.03
- added link camera_link_optical
- added link caster_wheel2, mass 0.1; collision sphere radius=0.08; visual sphere radius=0.08
Joints:
- added joint camera_joint: type fixed, parent chassis, child camera_link, origin xyz=0.005 0 0.1 rpy=0 0 0
- added joint camera_optical_joint: type fixed, parent camera_link, child camera_link_optical, origin xyz=0 0 0 rpy=-1.5707963267948966 0 -1.5707963267948966
- added joint caster_wheel_joint2: type fixed, parent chassis, child caster_wheel2, origin xyz=0.03 0 0
- joint chassis_joint: parent base_link -> botwheel
- joint left_wheel_joint: origin xyz=0 0.2425 0 rpy=-1.5707963267948966 0 0 -> xyz=-0.05 0.2425 0 rpy=-1.5707963267948966 0 0; parent base_link -> chassis
- joint right_wheel_joint: origin xyz=0 -0.2425 0 rpy=1.5707963267948966 0 0 -> xyz=-0.05 -0.2425 0 rpy=1.5707963267948966 0 0; parent base_link -> chassis

File: description/robot.urdf.xacro (robot description, xacro)
@@ -4,3 +4,4 @@
     <xacro:include filename="gazebo_control.xacro"/>
     <xacro:include filename="lidar.xacro"/>
+    <xacro:include filename="depth_camera.xacro"/>
 </robot>

File: description/robot_core.xacro (robot description, xacro)
@@ -18,9 +18,9 @@
     </material>
     <!-- Base Link-->
-    <link name="base_link">
+    <link name="botwheel">
     </link>
     <!-- Chassis Link -->
     <joint name="chassis_joint" type="fixed">
-        <parent link="base_link"/>
+        <parent link="botwheel"/>
         <child link="chassis"/>
         <origin xyz= "0.05 0 0"/>
@@ -46,7 +46,7 @@
     <!-- Left Wheel Link -->
     <joint name="left_wheel_joint" type="continuous">
-        <parent link="base_link"/>
+        <parent link="chassis"/>
         <child link="left_wheel"/>
-        <origin xyz= "0 0.2425 0" rpy="-${pi/2} 0 0"/>
+        <origin xyz= "-0.05 0.2425 0" rpy="-${pi/2} 0 0"/>
         <axis xyz="0 0 1"/>
     </joint>
@@ -57,4 +57,5 @@
             </geometry>
             <material name="black"/>
+            <origin xyz="0 0 0"/>
         </visual>
         <collision>
@@ -68,8 +69,8 @@
     </link>
      <!-- Right Wheel Link -->
-     <joint name="right_wheel_joint" type="continuous">
-        <parent link="base_link"/>
+    <joint name="right_wheel_joint" type="continuous">
+        <parent link="chassis"/>
         <child link="right_wheel"/>
-        <origin xyz= "0 -0.2425 0" rpy="${pi/2} 0 0"/>
+        <origin xyz= "-0.05 -0.2425 0" rpy="${pi/2} 0 0"/>
         <axis xyz="0 0 -1"/>
     </joint>
@@ -80,4 +81,5 @@
             </geometry>
             <material name="black"/>
+            <origin xyz="0 0 0"/>
         </visual>
         <collision>
@@ -116,3 +118,28 @@
         <mu2 value="0.0001"/>
     </gazebo>
+    <joint name="caster_wheel_joint2" type="fixed">
+        <parent link="chassis"/>
+        <child link="caster_wheel2"/>
+        <origin xyz="0.03 0 0"/>
+    </joint>
+    <link name="caster_wheel2">
+        <visual>
+            <geometry>
+                <sphere radius="0.08"/>
+            </geometry>
+            <material name="blue"/>
+        </visual>
+        <collision>
+            <geometry>
+                <sphere radius="0.08"/>
+            </geometry>
+        </collision>
+        <xacro:inertial_sphere mass="0.1" radius="0.05">
+            <origin xyz="0 0 0" rpy="0 0 0"/>
+        </xacro:inertial_sphere>
+    </link>
+    <gazebo reference="caster_wheel2">
+        <mu1 value="0.0001"/>
+        <mu2 value="0.0001"/>
+    </gazebo>
 </robot>
