Commit message: Finished Simulation

File: description/depth_camera.xacro (robot description, xacro)
@@ -21,5 +21,5 @@
     <link name="camera_link_optical">
     </link>
-    <gazebo reference="camera_link_optical">
+    <gazebo reference="camera_link">
         <material>Gazebo/Red</material>
         <sensor name="rgbd_camera" type="rgbd_camera">

File: description/gazebo_control.xacro (robot description, xacro)
@@ -27,5 +27,5 @@
             </input>
             <output type="gz.msgs.Twist" topic="/cmd_vel">
-            linear: {x: 3}, angular: {z: 0.0}
+            linear: {x: 5}, angular: {z: 0.0}
             </output>
         </plugin>
@@ -36,5 +36,5 @@
             </input>
             <output type="gz.msgs.Twist" topic="/cmd_vel">
-                linear: {x: -3}, angular: {z: 0.0}
+                linear: {x: -5}, angular: {z: 0.0}
             </output>
         </plugin>

File: description/robot.urdf.xacro (robot description, xacro)
@@ -2,5 +2,6 @@
 <robot xmlns:xacro="http://www.ros.org/wiki/xacro"  name="robot">
     <xacro:include filename="robot_core.xacro"/>
-    <xacro:include filename="gazebo_control.xacro"/>
+    <!-- <xacro:include filename="gazebo_control.xacro"/> -->
+    <xacro:include filename="ros2_control.xacro" />
     <xacro:include filename="lidar.xacro"/>
     <xacro:include filename="depth_camera.xacro"/>

File: description/robot_core.xacro (robot description, xacro)
@@ -19,4 +19,12 @@
     <!-- Base Link-->
     <link name="botwheel">
+    </link>
+    <!-- BASE_FOOTPRINT LINK -->
+    <joint name="base_footprint_joint" type="fixed">
+        <parent link="botwheel"/>
+        <child link="base_footprint"/>
+        <origin xyz="0 0 0" rpy="0 0 0"/>
+    </joint>
+    <link name="base_footprint">
     </link>
     <!-- Chassis Link -->
@@ -118,5 +126,5 @@
         <mu2 value="0.0001"/>
     </gazebo>
-    <joint name="caster_wheel_joint2" type="fixed">
+    <!-- <joint name="caster_wheel_joint2" type="fixed">
         <parent link="chassis"/>
         <child link="caster_wheel2"/>
@@ -142,4 +150,4 @@
         <mu1 value="0.0001"/>
         <mu2 value="0.0001"/>
-    </gazebo>
+    </gazebo> -->
 </robot>
