Commit message: Finalizing Launch Files

File: description/lidar.xacro (robot description, xacro)
@@ -16,5 +16,5 @@
             <geometry>
                 <cylinder radius="0.08" length="0.045"/>
-            </geometry>f
+            </geometry>
         </collision>
         <xacro:inertial_cylinder mass="0.15" length="0.04" radius="0.05">
