Commit message: Controller Config Update

File: description/botwheel_description.urdf.xacro (robot description, xacro)
@@ -69,5 +69,5 @@
         <parent link="chassis"/>
         <child link="left_wheel"/>
-        <origin xyz= "-0.05 0.2425 0" rpy="-${pi/2} 0 0"/>
+        <origin xyz= "-0.05 0.2425 0" rpy="${pi/2} 0 0"/>
         <axis xyz="0 0 1"/>
     </joint>
@@ -75,5 +75,5 @@
         <visual>
             <geometry>
-                <cylinder radius="0.08" length="0.045"/>
+                <cylinder radius="0.0855" length="0.045"/>
             </geometry>
             <material name="black"/>
@@ -82,5 +82,5 @@
         <collision>
             <geometry>
-                <cylinder radius="0.08" length="0.045"/>
+                <cylinder radius="0.0855" length="0.045"/>
             </geometry>
         </collision>
@@ -99,5 +99,5 @@
         <visual>
             <geometry>
-                <cylinder radius="0.08" length="0.045"/>
+                <cylinder radius="0.0855" length="0.045"/>
             </geometry>
             <material name="black"/>
@@ -106,5 +106,5 @@
         <collision>
             <geometry>
-                <cylinder radius="0.08" length="0.045"/>
+                <cylinder radius="0.0855" length="0.045"/>
             </geometry>
         </collision>
@@ -122,5 +122,5 @@
         <visual>
             <geometry>
-                <sphere radius="0.08"/>
+                <sphere radius="0.0855"/>
             </geometry>
             <material name="blue"/>
@@ -128,5 +128,5 @@
         <collision>
             <geometry>
-                <sphere radius="0.08"/>
+                <sphere radius="0.0855"/>
             </geometry>
         </collision>
@@ -142,5 +142,5 @@
         <parent link="chassis"/>
         <child link="laser"/>
-        <origin xyz="-0.095 0 0.145" rpy="0 0 0"/>
+        <origin xyz="-0.095 0 0.145" rpy="${pi} ${pi} 0"/>
     </joint>
     <link name="laser">
